File: eagle/projects/led.sch (EAGLE design)
At the start: 3 parts, among them X1 CLAMP_1X2-T-2.5MM

Commit message: added frame around layout
Parts:
- added R2: 330, be_rcl:R_S_0805
Connections:
- net GND: now also R2.2
- net LED_A: now also R2.1
Changed lines of the file:
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@@
 <?xml version="1.0" encoding="utf-8"?>
 <!DOCTYPE eagle SYSTEM "eagle.dtd">
-<eagle version="9.2.2">
+<eagle version="7.7.0">
 <drawing>
 <settings>
@@
 </part>
 <part name="GND2" library="be_supply" deviceset="GND" device=""/>
+<part name="R2" library="be_rcl" deviceset="R" device="_S_0805" value="330">
+<attribute name="PART_CODE_BEL" value="R_PAC_S_0805_VAL_330"/>
+</part>
+<part name="GND3" library="be_supply" deviceset="GND" device=""/>
 </parts>
 <sheets>
@@
 <attribute name="VALUE" x="176.022" y="41.275" size="1.27" layer="96" font="fixed"/>
 </instance>
+<instance part="R2" gate="G$1" x="205.74" y="68.58" smashed="yes">
+<attribute name="NAME" x="203.2" y="72.39" size="1.27" layer="95" font="fixed"/>
+<attribute name="VALUE" x="203.2" y="70.485" size="1.27" layer="96" font="fixed"/>
+</instance>
+<instance part="GND3" gate="1" x="213.36" y="43.18" smashed="yes">
+<attribute name="VALUE" x="211.582" y="41.275" size="1.27" layer="96" font="fixed"/>
+</instance>
 </instances>
 <busses>
@@
 <wire x1="190.5" y1="68.58" x2="195.58" y2="68.58" width="0.1524" layer="91"/>
 <wire x1="195.58" y1="68.58" x2="195.58" y2="55.88" width="0.1524" layer="91"/>
+<pinref part="R2" gate="G$1" pin="1"/>
+<wire x1="200.66" y1="68.58" x2="195.58" y2="68.58" width="0.1524" layer="91"/>
+<junction x="195.58" y="68.58"/>
 </segment>
 </net>
@@
 <pinref part="GND2" gate="1" pin="GND"/>
 </segment>
+<segment>
+<pinref part="R2" gate="G$1" pin="2"/>
+<wire x1="210.82" y1="68.58" x2="213.36" y2="68.58" width="0.1524" layer="91"/>
+<wire x1="213.36" y1="68.58" x2="213.36" y2="45.72" width="0.1524" layer="91"/>
+<pinref part="GND3" gate="1" pin="GND"/>
+</segment>
 </net>

Commit message: test attributes
Parts:
- R1: TRM (none) -> 0.123
Changed lines of the file:
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@@
 <part name="R1" library="be_rcl" deviceset="R" device="_S_0805" value="330">
 <attribute name="PART_CODE_BEL" value="R_PAC_S_0805_VAL_330"/>
+<attribute name="TRM" value="0.123"/>
 </part>
 <part name="GND2" library="be_supply" deviceset="GND" device=""/>
@@
 <attribute name="NAME" x="182.88" y="72.39" size="1.27" layer="95" font="fixed"/>
 <attribute name="VALUE" x="182.88" y="70.485" size="1.27" layer="96" font="fixed"/>
+<attribute name="TRM" x="185.42" y="68.58" size="1.27" layer="96" font="fixed" display="off"/>
 </instance>
 <instance part="GND2" gate="1" x="177.8" y="43.18" smashed="yes">

Commit message: remove attribute trm
Parts:
- R1: TRM 0.123 -> (none)
Changed lines of the file:
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@@
 <?xml version="1.0" encoding="utf-8"?>
 <!DOCTYPE eagle SYSTEM "eagle.dtd">
-<eagle version="7.7.0">
+<eagle version="9.5.2">
 <drawing>
 <settings>
 <setting alwaysvectorfont="no"/>
+<setting keepoldvectorfont="yes"/>
 <setting verticaltext="up"/>
 </settings>
@@
 <part name="R1" library="be_rcl" deviceset="R" device="_S_0805" value="330">
 <attribute name="PART_CODE_BEL" value="R_PAC_S_0805_VAL_330"/>
-<attribute name="TRM" value="0.123"/>
 </part>
 <part name="GND2" library="be_supply" deviceset="GND" device=""/>
@@
 <attribute name="NAME" x="182.88" y="72.39" size="1.27" layer="95" font="fixed"/>
 <attribute name="VALUE" x="182.88" y="70.485" size="1.27" layer="96" font="fixed"/>
-<attribute name="TRM" x="185.42" y="68.58" size="1.27" layer="96" font="fixed" display="off"/>
 </instance>
 <instance part="GND2" gate="1" x="177.8" y="43.18" smashed="yes">
